Commit message: feat: Add wheels and joints to robot

File: urdf/my_robot.xacro (robot description, xacro)
@@ -55,3 +55,65 @@
     </visual>
   </link>
+  <link name="right_wheel">
+    <collision name="right_wheel_collision">
+      <origin xyz='0 0 0' rpy='0 1.5707 1.5707'/>
+      <geometry>
+        <cylinder radius='0.1' length='0.05'/>
+      </geometry>
+    </collision>
+    <inertial name="right_wheel_intertial">
+      <mass value="5.0"/>
+      <origin xyz="0.0 0 0" rpy=" 0 1.5707 1.5707"/>
+      <inertia
+          ixx="0.1" ixy="0" ixz="0"
+          iyy="0.1" iyz="0"
+          izz="0.1"
+      />
+    </inertial>
+    <visual name="right_wheel_visual">
+      <origin xyz='0 0 0' rpy='0 1.5707 1.5707'/>
+      <geometry>
+        <cylinder radius='0.1' length='0.05'/>
+      </geometry>
+    </visual>
+  </link>
+  <link name="left_wheel">
+    <collision name="left_wheel_collision">
+      <origin xyz='0 0 0' rpy='0 1.5707 1.5707'/>
+      <geometry>
+        <cylinder radius='0.1' length='0.05'/>
+      </geometry>
+    </collision>
+    <inertial name="left_wheel_intertial">
+      <mass value="5.0"/>
+      <origin xyz="0.0 0 0" rpy=" 0 1.5707 1.5707"/>
+      <inertia
+          ixx="0.1" ixy="0" ixz="0"
+          iyy="0.1" iyz="0"
+          izz="0.1"
+      />
+    </inertial>
+    <visual name="left_wheel_visual">
+      <origin xyz='0 0 0' rpy='0 1.5707 1.5707'/>
+      <geometry>
+        <cylinder radius='0.1' length='0.05'/>
+      </geometry>
+    </visual>
+  </link>
+  <joint type="continuous" name="left_wheel_hinge">
+   <origin xyz="0 0.15 0" rpy="0 0 0"/>
+   <child link="left_wheel"/>
+   <parent link="chassis"/>
+   <axis xyz="0 1 0" rpy="0 0 0"/>
+   <limit effort="10000" velocity="1000"/>
+   <dynamics damping="1.0" friction="1.0"/>
+ </joint>
+ <joint type="continuous" name="right_wheel_hinge">
+   <origin xyz="0 -0.15 0" rpy="0 0 0"/>
+   <child link="right_wheel"/>
+   <parent link="chassis"/>
+   <axis xyz="0 1 0" rpy="0 0 0"/>
+   <limit effort="10000" velocity="1000"/>
+   <dynamics damping="1.0" friction="1.0"/>
+ </joint>
 </robot>

Commit message: feat: Add sensors to robot
Box for a camera and Lidar as a mesh.

File: urdf/my_robot.xacro (robot description, xacro)
@@ -117,3 +117,60 @@
    <dynamics damping="1.0" friction="1.0"/>
  </joint>
+ <link name='camera'>
+   <collision name="camera_collision">
+     <origin xyz='0 0 0' rpy='0 0 0'/>
+     <geometry>
+       <box size=".05 .05 .05"/>
+     </geometry>
+   </collision>
+   <inertial name="camera_intertial">
+     <mass value="0.1"/>
+     <origin xyz="0.05 0.05 0.05"/>
+     <inertia
+         ixx="1e-6" ixy="0" ixz="0"
+         iyy="1e-6" iyz="0"
+         izz="1e-6"
+     />
+   </inertial>
+   <visual name="camera_visual">
+     <origin xyz='0 0 0' rpy='0 0 0'/>
+     <geometry>
+       <box size='0.05 0.05 0.05'/>
+     </geometry>
+   </visual>
+ </link>
+ <joint type='fixed' name='camera_joint'>
+   <origin xyz='0.2 0 0' rpy='0 0 0'/>
+   <child link='camera'/>
+   <parent link='chassis'/>
+   <axis xyz='0 1 0'/>
+ </joint>
+ <link name='hokuyo'>
+   <collision name="hokuyo_collision">
+     <origin xyz='0 0 0' rpy='0 0 0'/>
+     <geometry>
+       <box size=".1 .1 .1"/>
+     </geometry>
+   </collision>
+   <inertial name="hokuyo_intertial">
+     <mass value="1e-5"/>
+     <inertia
+          ixx="1e-6" ixy="0" ixz="0"
+          iyy="1e-6" iyz="0"
+          izz="1e-6"
+     />
+   </inertial>
+   <visual name="hokuyo_visual">
+     <origin xyz='0 0 0' rpy='0 0 0'/>
+     <geometry>
+       <mesh filename='package://my_robot/meshes/hokuyo.dae'/>
+     </geometry>
+   </visual>
+ </link>
+ <joint type='fixed' name='hokuyo_joint'>
+   <origin xyz='0.15 0 0.1' rpy='0 0 0'/>
+   <child link='hokuyo'/>
+   <parent link='chassis'/>
+   <axis xyz='0 1 0'/>
+ </joint>
 </robot>

Commit message: feat: improve wheels

File: urdf/my_robot.xacro (robot description, xacro)
@@ -78,4 +78,10 @@
       </geometry>
     </visual>
+    <visual name="right_rin_visual">
+      <origin xyz='0 -0.025 0' rpy='0 1.5707 1.5707'/>
+      <geometry>
+        <cylinder radius='0.03' length='0.05'/>
+      </geometry>
+    </visual>
   </link>
   <link name="left_wheel">
@@ -99,4 +105,10 @@
       <geometry>
         <cylinder radius='0.1' length='0.05'/>
+      </geometry>
+    </visual>
+    <visual name="left_rin_visual">
+      <origin xyz='0 0.025 0' rpy='0 1.5707 1.5707'/>
+      <geometry>
+        <cylinder radius='0.03' length='0.05'/>
       </geometry>
     </visual>

Commit message: feat: modify robot chassis

File: urdf/my_robot.xacro (robot description, xacro)
@@ -3,4 +3,7 @@
   <xacro:include filename="$(find my_robot)/urdf/my_robot.gazebo" />
   <link name="robot_footprint"></link>
+  <gazebo reference="chassis">
+    <material>Gazebo/Green</material>
+  </gazebo>
   <joint name="robot_footprint_joint" type="fixed">
     <origin xyz="0 0 0" rpy="0 0 0" />
@@ -55,4 +58,16 @@
       </geometry>
     </visual>
+    <visual name='passenger_case_visual'>
+      <origin xyz="-0.05 0 0.1" rpy=" 0 0 0"/>
+      <geometry>
+        <box size=".2 .15 .1"/>
+      </geometry>
+    </visual>
+    <visual name='top_decoration'>
+      <origin xyz="0 0 0.15" rpy=" 0 0 0"/>
+      <geometry>
+        <cylinder radius="0.025" length='0.05'/>
+      </geometry>
+    </visual>
   </link>
   <link name="right_wheel">

Commit message: chore: Add map of world and map.yml

File: urdf/my_robot.xacro (robot description, xacro)
@@ -5,4 +5,10 @@
   <gazebo reference="chassis">
     <material>Gazebo/Green</material>
+  </gazebo>
+  <gazebo reference="right_wheel">
+    <material>Gazebo/Black</material>
+  </gazebo>
+  <gazebo reference="left_wheel">
+    <material>Gazebo/Black</material>
   </gazebo>
   <joint name="robot_footprint_joint" type="fixed">

Commit message: feat: Add mapping node with default values

File: urdf/my_robot.xacro (robot description, xacro)
@@ -180,4 +180,11 @@
    <axis xyz='0 1 0'/>
  </joint>
+ <link name="camera_link_optical">
+ </link>
+ <joint name="camera_optical_joint" type="fixed">
+   <origin xyz="0 0 0" rpy="-1.5707 0 -1.5707"/>
+   <parent link="camera"/>
+   <child link="camera_link_optical"/>
+ </joint>
  <link name='hokuyo'>
    <collision name="hokuyo_collision">
